File: accuphase_e202_rectifier.sch (EAGLE design)
At the start: 12 parts

Commit message: added pcb
Parts:
- added H1, H2: MOUNT-PAD-ROUND3.0, holes:MOUNT-PAD-ROUND3.0
- D1, D2, D3, D4: value MUR820 -> MUR810; device diode:MUR820 -> diode:MUR810
Changed lines of the file:
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@@
 </classes>
 <parts>
-<part name="D1" library="diode" deviceset="MUR820" device=""/>
-<part name="D2" library="diode" deviceset="MUR820" device=""/>
-<part name="D3" library="diode" deviceset="MUR820" device=""/>
-<part name="D4" library="diode" deviceset="MUR820" device=""/>
 <part name="C1" library="resistor" deviceset="C-EU" device="075-032X103"/>
 <part name="C2" library="resistor" deviceset="C-EU" device="075-032X103"/>
@@
 <part name="VEE" library="wirepad" deviceset="3,81/1,4" device=""/>
 <part name="VCC" library="wirepad" deviceset="3,81/1,4" device=""/>
+<part name="H1" library="holes" deviceset="MOUNT-PAD-ROUND" device="3.0"/>
+<part name="H2" library="holes" deviceset="MOUNT-PAD-ROUND" device="3.0"/>
+<part name="D1" library="diode" deviceset="MUR810" device=""/>
+<part name="D2" library="diode" deviceset="MUR810" device=""/>
+<part name="D3" library="diode" deviceset="MUR810" device=""/>
+<part name="D4" library="diode" deviceset="MUR810" device=""/>
 </parts>
 <sheets>
@@
 </plain>
 <instances>
-<instance part="D1" gate="1" x="58.42" y="66.04"/>
-<instance part="D2" gate="1" x="73.66" y="55.88" rot="R270"/>
-<instance part="D3" gate="1" x="58.42" y="43.18"/>
-<instance part="D4" gate="1" x="48.26" y="55.88" rot="R270"/>
 <instance part="C1" gate="G$1" x="55.88" y="73.66" rot="R90"/>
 <instance part="C2" gate="G$1" x="81.28" y="55.88" rot="R180"/>
@@
 <instance part="VEE" gate="1" x="38.1" y="66.04"/>
 <instance part="VCC" gate="1" x="83.82" y="43.18" rot="R180"/>
+<instance part="H1" gate="G$1" x="30.48" y="91.44"/>
+<instance part="H2" gate="G$1" x="76.2" y="91.44"/>
+<instance part="D1" gate="1" x="58.42" y="66.04"/>
+<instance part="D2" gate="1" x="73.66" y="55.88" rot="R270"/>
+<instance part="D3" gate="1" x="58.42" y="43.18"/>
+<instance part="D4" gate="1" x="48.26" y="55.88" rot="R270"/>
 </instances>
 <busses>
@@
 <net name="N$1" class="0">
 <segment>
-<pinref part="D2" gate="1" pin="A"/>
 <wire x1="63.5" y1="66.04" x2="73.66" y2="66.04" width="0.1524" layer="91"/>
 <wire x1="73.66" y1="66.04" x2="73.66" y2="60.96" width="0.1524" layer="91"/>
@@
 <wire x1="60.96" y1="73.66" x2="63.5" y2="73.66" width="0.1524" layer="91"/>
 <wire x1="63.5" y1="73.66" x2="63.5" y2="66.04" width="0.1524" layer="91"/>
-<pinref part="D1" gate="1" pin="C"/>
 <wire x1="63.5" y1="66.04" x2="60.96" y2="66.04" width="0.1524" layer="91"/>
 <junction x="63.5" y="66.04"/>
@@
 <wire x1="73.66" y1="73.66" x2="73.66" y2="66.04" width="0.1524" layer="91"/>
 <junction x="73.66" y="66.04"/>
+<pinref part="D1" gate="1" pin="C"/>
+<pinref part="D2" gate="1" pin="A"/>
 </segment>
 </net>
@@
 <wire x1="73.66" y1="50.8" x2="73.66" y2="43.18" width="0.1524" layer="91"/>
 <wire x1="73.66" y1="43.18" x2="63.5" y2="43.18" width="0.1524" layer="91"/>
-<pinref part="D3" gate="1" pin="C"/>
 <pinref part="C2" gate="G$1" pin="1"/>
 <wire x1="63.5" y1="43.18" x2="60.96" y2="43.18" width="0.1524" layer="91"/>
 <wire x1="81.28" y1="53.34" x2="81.28" y2="50.8" width="0.1524" layer="91"/>
 <wire x1="81.28" y1="50.8" x2="73.66" y2="50.8" width="0.1524" layer="91"/>
-<pinref part="D2" gate="1" pin="C"/>
 <wire x1="73.66" y1="50.8" x2="73.66" y2="53.34" width="0.1524" layer="91"/>
 <junction x="73.66" y="50.8"/>
@@
 <wire x1="81.28" y1="43.18" x2="73.66" y2="43.18" width="0.1524" layer="91"/>
 <junction x="73.66" y="43.18"/>
+<pinref part="D2" gate="1" pin="C"/>
+<pinref part="D3" gate="1" pin="C"/>
 </segment>
 </net>
 <net name="N$3" class="0">
 <segment>
-<pinref part="D3" gate="1" pin="A"/>
-<pinref part="D4" gate="1" pin="C"/>
 <wire x1="55.88" y1="43.18" x2="53.34" y2="43.18" width="0.1524" layer="91"/>
 <wire x1="53.34" y1="43.18" x2="48.26" y2="43.18" width="0.1524" layer="91"/>
@@
 <wire x1="48.26" y1="35.56" x2="48.26" y2="43.18" width="0.1524" layer="91"/>
 <junction x="48.26" y="43.18"/>
+<pinref part="D3" gate="1" pin="A"/>
+<pinref part="D4" gate="1" pin="C"/>
 </segment>
 </net>
 <net name="N$4" class="0">
 <segment>
-<pinref part="D4" gate="1" pin="A"/>
-<pinref part="D1" gate="1" pin="A"/>
 <wire x1="48.26" y1="58.42" x2="48.26" y2="60.96" width="0.1524" layer="91"/>
 <wire x1="48.26" y1="60.96" x2="48.26" y2="66.04" width="0.1524" layer="91"/>
@@
 <wire x1="40.64" y1="66.04" x2="48.26" y2="66.04" width="0.1524" layer="91"/>
 <junction x="48.26" y="66.04"/>
+<pinref part="D1" gate="1" pin="A"/>
+<pinref part="D4" gate="1" pin="A"/>
 </segment>
 </net>
