File: accuphase_e202_rectifier.brd (EAGLE design)
At the start: 78.7 x 31.4 mm, 14 parts

Commit message: minor improvement
Parts:
- moved AC1 20.3 mm to (19.1, 3.81)
- moved VCC 18.2 mm to (39.4, 3.81)
- moved VEE 6.84 mm to (19.1, 14.0)
Routing:
- net N$1: track 82.6 -> 62.2 mm
- net N$4: track 102.4 -> 95.0 mm
- net N$2: track 59.7 -> 62.2 mm
- added copper zone on layer 16, net N$5
Changed lines of the file:
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@@
 <layer number="27" name="tValues" color="7" fill="1" visible="yes" active="yes"/>
 <layer number="28" name="bValues" color="7" fill="1" visible="yes" active="yes"/>
-<layer number="29" name="tStop" color="7" fill="3" visible="no" active="yes"/>
-<layer number="30" name="bStop" color="7" fill="6" visible="no" active="yes"/>
-<layer number="31" name="tCream" color="7" fill="4" visible="no" active="yes"/>
-<layer number="32" name="bCream" color="7" fill="5" visible="no" active="yes"/>
-<layer number="33" name="tFinish" color="6" fill="3" visible="no" active="yes"/>
-<layer number="34" name="bFinish" color="6" fill="6" visible="no" active="yes"/>
-<layer number="35" name="tGlue" color="7" fill="4" visible="no" active="yes"/>
-<layer number="36" name="bGlue" color="7" fill="5" visible="no" active="yes"/>
-<layer number="37" name="tTest" color="7" fill="1" visible="no" active="yes"/>
-<layer number="38" name="bTest" color="7" fill="1" visible="no" active="yes"/>
+<layer number="29" name="tStop" color="7" fill="3" visible="yes" active="yes"/>
+<layer number="30" name="bStop" color="7" fill="6" visible="yes" active="yes"/>
+<layer number="31" name="tCream" color="7" fill="4" visible="yes" active="yes"/>
+<layer number="32" name="bCream" color="7" fill="5" visible="yes" active="yes"/>
+<layer number="33" name="tFinish" color="6" fill="3" visible="yes" active="yes"/>
+<layer number="34" name="bFinish" color="6" fill="6" visible="yes" active="yes"/>
+<layer number="35" name="tGlue" color="7" fill="4" visible="yes" active="yes"/>
+<layer number="36" name="bGlue" color="7" fill="5" visible="yes" active="yes"/>
+<layer number="37" name="tTest" color="7" fill="1" visible="yes" active="yes"/>
+<layer number="38" name="bTest" color="7" fill="1" visible="yes" active="yes"/>
 <layer number="39" name="tKeepout" color="4" fill="11" visible="yes" active="yes"/>
 <layer number="40" name="bKeepout" color="1" fill="11" visible="yes" active="yes"/>
@@
 <layer number="42" name="bRestrict" color="1" fill="10" visible="yes" active="yes"/>
 <layer number="43" name="vRestrict" color="2" fill="10" visible="yes" active="yes"/>
-<layer number="44" name="Drills" color="7" fill="1" visible="no" active="yes"/>
-<layer number="45" name="Holes" color="7" fill="1" visible="no" active="yes"/>
-<layer number="46" name="Milling" color="3" fill="1" visible="no" active="yes"/>
-<layer number="47" name="Measures" color="7" fill="1" visible="no" active="yes"/>
+<layer number="44" name="Drills" color="7" fill="1" visible="yes" active="yes"/>
+<layer number="45" name="Holes" color="7" fill="1" visible="yes" active="yes"/>
+<layer number="46" name="Milling" color="3" fill="1" visible="yes" active="yes"/>
+<layer number="47" name="Measures" color="7" fill="1" visible="yes" active="yes"/>
 <layer number="48" name="Document" color="7" fill="1" visible="yes" active="yes"/>
 <layer number="49" name="Reference" color="7" fill="1" visible="yes" active="yes"/>
@@
 </autorouter>
 <elements>
-<element name="AC1" library="wirepad" package="3,81/1,4" value="" x="39.37" y="3.81"/>
+<element name="AC1" library="wirepad" package="3,81/1,4" value="" x="19.05" y="3.81"/>
 <element name="AC2" library="wirepad" package="3,81/1,4" value="" x="59.69" y="3.81"/>
 <element name="C1" library="resistor" package="C075-032X103" value="" x="8.89" y="10.16" rot="R180"/>
@@
 <element name="C3" library="resistor" package="C075-032X103" value="" x="49.53" y="10.16"/>
 <element name="C4" library="resistor" package="C075-032X103" value="" x="69.85" y="10.16" rot="R180"/>
-<element name="VCC" library="wirepad" package="3,81/1,4" value="" x="21.59" y="7.62"/>
-<element name="VEE" library="wirepad" package="3,81/1,4" value="" x="16.51" y="7.62"/>
+<element name="VCC" library="wirepad" package="3,81/1,4" value="" x="39.37" y="3.81"/>
+<element name="VEE" library="wirepad" package="3,81/1,4" value="" x="19.05" y="13.97"/>
 <element name="H1" library="holes" package="3,0-PAD" value="MOUNT-PAD-ROUND3.0" x="73.66" y="26.67"/>
 <element name="H2" library="holes" package="3,0-PAD" value="MOUNT-PAD-ROUND3.0" x="5.08" y="26.67"/>
@@
 <wire x1="31.75" y1="17.78" x2="33.02" y2="17.78" width="2.54" layer="16"/>
 <wire x1="33.02" y1="17.78" x2="33.02" y2="10.16" width="2.54" layer="16"/>
-<wire x1="39.37" y1="3.81" x2="39.37" y2="17.78" width="2.54" layer="16"/>
-<wire x1="39.37" y1="17.78" x2="31.75" y2="17.78" width="2.54" layer="16"/>
 <wire x1="6.35" y1="17.78" x2="5.08" y2="17.78" width="2.54" layer="16"/>
 <wire x1="5.08" y1="17.78" x2="5.08" y2="10.16" width="2.54" layer="16"/>
 <wire x1="5.08" y1="10.16" x2="5.08" y2="2.54" width="2.54" layer="16"/>
-<wire x1="5.08" y1="2.54" x2="33.02" y2="2.54" width="2.54" layer="16"/>
+<wire x1="5.08" y1="2.54" x2="19.05" y2="2.54" width="2.54" layer="16"/>
+<wire x1="19.05" y1="2.54" x2="33.02" y2="2.54" width="2.54" layer="16"/>
 <wire x1="33.02" y1="2.54" x2="33.02" y2="10.16" width="2.54" layer="16"/>
+<wire x1="19.05" y1="3.81" x2="19.05" y2="2.54" width="2.54" layer="16"/>
 </signal>
 <signal name="N$2">
@@
 <wire x1="45.72" y1="10.16" x2="45.72" y2="17.78" width="2.54" layer="16"/>
 <wire x1="45.72" y1="17.78" x2="46.99" y2="17.78" width="2.54" layer="16"/>
-<wire x1="21.59" y1="17.78" x2="26.67" y2="17.78" width="2.54" layer="16"/>
 <wire x1="45.72" y1="17.78" x2="45.72" y2="21.59" width="2.54" layer="16"/>
-<wire x1="45.72" y1="21.59" x2="26.67" y2="21.59" width="2.54" layer="16"/>
+<wire x1="45.72" y1="21.59" x2="39.37" y2="21.59" width="2.54" layer="16"/>
+<wire x1="39.37" y1="21.59" x2="26.67" y2="21.59" width="2.54" layer="16"/>
 <wire x1="26.67" y1="21.59" x2="26.67" y2="17.78" width="2.54" layer="16"/>
-<wire x1="21.59" y1="17.78" x2="21.59" y2="7.62" width="2.54" layer="16"/>
+<wire x1="39.37" y1="3.81" x2="39.37" y2="21.59" width="2.54" layer="16"/>
 </signal>
 <signal name="N$3">
@@
 <wire x1="72.39" y1="17.78" x2="73.66" y2="17.78" width="2.54" layer="16"/>
 <wire x1="73.66" y1="17.78" x2="73.66" y2="10.16" width="2.54" layer="16"/>
-<wire x1="16.51" y1="17.78" x2="16.51" y2="7.62" width="2.54" layer="16"/>
+<wire x1="16.51" y1="17.78" x2="19.05" y2="13.97" width="2.54" layer="16"/>
 <wire x1="16.51" y1="17.78" x2="16.51" y2="25.4" width="2.54" layer="16"/>
-<wire x1="16.51" y1="25.4" x2="62.23" y2="25.4" width="2.54" layer="16"/>
-<wire x1="62.23" y1="25.4" x2="62.23" y2="21.59" width="2.54" layer="16"/>
-<wire x1="62.23" y1="21.59" x2="69.85" y2="21.59" width="2.54" layer="16"/>
-<wire x1="69.85" y1="21.59" x2="72.39" y2="17.78" width="2.54" layer="16"/>
+<wire x1="16.51" y1="25.4" x2="67.31" y2="25.4" width="2.54" layer="16"/>
+<wire x1="67.31" y1="25.4" x2="72.39" y2="17.78" width="2.54" layer="16"/>
+</signal>
+<signal name="N$5">
+<polygon width="1.27" layer="16">
+<vertex x="0" y="0"/>
+<vertex x="0" y="31.75"/>
+<vertex x="78.74" y="31.75"/>
+<vertex x="78.74" y="0"/>
+</polygon>
 </signal>
 </signals>
